Commit message: feat: add option for abs path

File: robotiq_description/urdf/robotiq_2f_85_macro.urdf.xacro (robot description, xacro)
@@ -8,4 +8,5 @@
         sim_gazebo:=false
         sim_isaac:=false
+        force_abs_paths:=false
         isaac_joint_commands:=/isaac_joint_commands
         isaac_joint_states:=/isaac_joint_states
@@ -31,10 +32,20 @@
             <visual>
                 <geometry>
-                    <mesh filename="package://robotiq_description/meshes/visual/2f_85/robotiq_base.dae" />
-                </geometry>
-            </visual>
-            <collision>
-                <geometry>
-                    <mesh filename="package://robotiq_description/meshes/collision/2f_85/robotiq_base.stl" />
+                    <xacro:unless value="${force_abs_paths}">
+                        <mesh filename="package://robotiq_description/meshes/visual/2f_85/robotiq_base.dae" />
+                    </xacro:unless>
+                    <xacro:if value="${force_abs_paths}">
+                        <mesh filename="file://$(find robotiq_description)/meshes/visual/2f_85/robotiq_base.dae" />
+                    </xacro:if>
+                </geometry>
+            </visual>
+            <collision>
+                <geometry>
+                    <xacro:unless value="${force_abs_paths}">
+                        <mesh filename="package://robotiq_description/meshes/collision/2f_85/robotiq_base.stl" />
+                    </xacro:unless>
+                    <xacro:if value="${force_abs_paths}">
+                        <mesh filename="file://$(find robotiq_description)/meshes/collision/2f_85/robotiq_base.stl" />
+                    </xacro:if>
                 </geometry>
             </collision>
@@ -48,10 +59,20 @@
             <visual>
                 <geometry>
-                    <mesh filename="package://robotiq_description/meshes/visual/2f_85/left_knuckle.dae" />
-                </geometry>
-            </visual>
-            <collision>
-                <geometry>
-                    <mesh filename="package://robotiq_description/meshes/collision/2f_85/left_knuckle.stl" />
+                    <xacro:unless value="${force_abs_paths}">
+                        <mesh filename="package://robotiq_description/meshes/visual/2f_85/left_knuckle.dae" />
+                    </xacro:unless>
+                    <xacro:if value="${force_abs_paths}">
+                        <mesh filename="file://$(find robotiq_description)/meshes/visual/2f_85/left_knuckle.dae" />
+                    </xacro:if>
+                </geometry>
+            </visual>
+            <collision>
+                <geometry>
+                    <xacro:unless value="${force_abs_paths}">
+                        <mesh filename="package://robotiq_description/meshes/collision/2f_85/left_knuckle.stl" />
+                    </xacro:unless>
+                    <xacro:if value="${force_abs_paths}">
+                        <mesh filename="file://$(find robotiq_description)/meshes/collision/2f_85/left_knuckle.stl" />
+                    </xacro:if>
                 </geometry>
             </collision>
@@ -65,10 +86,20 @@
             <visual>
                 <geometry>
-                    <mesh filename="package://robotiq_description/meshes/visual/2f_85/right_knuckle.dae" />
-                </geometry>
-            </visual>
-            <collision>
-                <geometry>
-                    <mesh filename="package://robotiq_description/meshes/collision/2f_85/right_knuckle.stl" />
+                    <xacro:unless value="${force_abs_paths}">
+                        <mesh filename="package://robotiq_description/meshes/visual/2f_85/right_knuckle.dae" />
+                    </xacro:unless>
+                    <xacro:if value="${force_abs_paths}">
+                        <mesh filename="file://$(find robotiq_description)/meshes/visual/2f_85/right_knuckle.dae" />
+                    </xacro:if>
+                </geometry>
+            </visual>
+            <collision>
+                <geometry>
+                    <xacro:unless value="${force_abs_paths}">
+                        <mesh filename="package://robotiq_description/meshes/collision/2f_85/right_knuckle.stl" />
+                    </xacro:unless>
+                    <xacro:if value="${force_abs_paths}">
+                        <mesh filename="file://$(find robotiq_description)/meshes/collision/2f_85/right_knuckle.stl" />
+                    </xacro:if>
                 </geometry>
             </collision>
@@ -82,10 +113,20 @@
             <visual>
                 <geometry>
-                    <mesh filename="package://robotiq_description/meshes/visual/2f_85/left_finger.dae" />
-                </geometry>
-            </visual>
-            <collision>
-                <geometry>
-                    <mesh filename="package://robotiq_description/meshes/collision/2f_85/left_finger.stl" />
+                    <xacro:unless value="${force_abs_paths}">
+                        <mesh filename="package://robotiq_description/meshes/visual/2f_85/left_finger.dae" />
+                    </xacro:unless>
+                    <xacro:if value="${force_abs_paths}">
+                        <mesh filename="file://$(find robotiq_description)/meshes/visual/2f_85/left_finger.dae" />
+                    </xacro:if>
+                </geometry>
+            </visual>
+            <collision>
+                <geometry>
+                    <xacro:unless value="${force_abs_paths}">
+                        <mesh filename="package://robotiq_description/meshes/collision/2f_85/left_finger.stl" />
+                    </xacro:unless>
+                    <xacro:if value="${force_abs_paths}">
+                        <mesh filename="file://$(find robotiq_description)/meshes/collision/2f_85/left_finger.stl" />
+                    </xacro:if>
                 </geometry>
             </collision>
@@ -99,10 +140,20 @@
             <visual>
                 <geometry>
-                    <mesh filename="package://robotiq_description/meshes/visual/2f_85/right_finger.dae" />
-                </geometry>
-            </visual>
-            <collision>
-                <geometry>
-                    <mesh filename="package://robotiq_description/meshes/collision/2f_85/right_finger.stl" />
+                    <xacro:unless value="${force_abs_paths}">
+                        <mesh filename="package://robotiq_description/meshes/visual/2f_85/right_finger.dae" />
+                    </xacro:unless>
+                    <xacro:if value="${force_abs_paths}">
+                        <mesh filename="file://$(find robotiq_description)/meshes/visual/2f_85/right_finger.dae" />
+                    </xacro:if>
+                </geometry>
+            </visual>
+            <collision>
+                <geometry>
+                    <xacro:unless value="${force_abs_paths}">
+                        <mesh filename="package://robotiq_description/meshes/collision/2f_85/right_finger.stl" />
+                    </xacro:unless>
+                    <xacro:if value="${force_abs_paths}">
+                        <mesh filename="file://$(find robotiq_description)/meshes/collision/2f_85/right_finger.stl" />
+                    </xacro:if>
                 </geometry>
             </collision>
@@ -116,10 +167,20 @@
             <visual>
                 <geometry>
-                    <mesh filename="package://robotiq_description/meshes/visual/2f_85/left_inner_knuckle.dae" />
-                </geometry>
-            </visual>
-            <collision>
-                <geometry>
-                    <mesh filename="package://robotiq_description/meshes/collision/2f_85/left_inner_knuckle.stl" />
+                    <xacro:unless value="${force_abs_paths}">
+                        <mesh filename="package://robotiq_description/meshes/visual/2f_85/left_inner_knuckle.dae" />
+                    </xacro:unless>
+                    <xacro:if value="${force_abs_paths}">
+                        <mesh filename="file://$(find robotiq_description)/meshes/visual/2f_85/left_inner_knuckle.dae" />
+                    </xacro:if>
+                </geometry>
+            </visual>
+            <collision>
+                <geometry>
+                    <xacro:unless value="${force_abs_paths}">
+                        <mesh filename="package://robotiq_description/meshes/collision/2f_85/left_inner_knuckle.stl" />
+                    </xacro:unless>
+                    <xacro:if value="${force_abs_paths}">
+                        <mesh filename="file://$(find robotiq_description)/meshes/collision/2f_85/left_inner_knuckle.stl" />
+                    </xacro:if>
                 </geometry>
             </collision>
@@ -133,10 +194,20 @@
             <visual>
                 <geometry>
-                    <mesh filename="package://robotiq_description/meshes/visual/2f_85/right_inner_knuckle.dae" />
-                </geometry>
-            </visual>
-            <collision>
-                <geometry>
-                    <mesh filename="package://robotiq_description/meshes/collision/2f_85/right_inner_knuckle.stl" />
+                    <xacro:unless value="${force_abs_paths}">
+                        <mesh filename="package://robotiq_description/meshes/visual/2f_85/right_inner_knuckle.dae" />
+                    </xacro:unless>
+                    <xacro:if value="${force_abs_paths}">
+                        <mesh filename="file://$(find robotiq_description)/meshes/visual/2f_85/right_inner_knuckle.dae" />
+                    </xacro:if>
+                </geometry>
+            </visual>
+            <collision>
+                <geometry>
+                    <xacro:unless value="${force_abs_paths}">
+                        <mesh filename="package://robotiq_description/meshes/collision/2f_85/right_inner_knuckle.stl" />
+                    </xacro:unless>
+                    <xacro:if value="${force_abs_paths}">
+                        <mesh filename="file://$(find robotiq_description)/meshes/collision/2f_85/right_inner_knuckle.stl" />
+                    </xacro:if>
                 </geometry>
             </collision>
@@ -150,10 +221,20 @@
             <visual>
                 <geometry>
-                    <mesh filename="package://robotiq_description/meshes/visual/2f_85/left_finger_tip.dae" />
-                </geometry>
-            </visual>
-            <collision>
-                <geometry>
-                    <mesh filename="package://robotiq_description/meshes/collision/2f_85/left_finger_tip.stl" />
+                    <xacro:unless value="${force_abs_paths}">
+                        <mesh filename="package://robotiq_description/meshes/visual/2f_85/left_finger_tip.dae" />
+                    </xacro:unless>
+                    <xacro:if value="${force_abs_paths}">
+                        <mesh filename="file://$(find robotiq_description)/meshes/visual/2f_85/left_finger_tip.dae" />
+                    </xacro:if>
+                </geometry>
+            </visual>
+            <collision>
+                <geometry>
+                    <xacro:unless value="${force_abs_paths}">
+                        <mesh filename="package://robotiq_description/meshes/collision/2f_85/left_finger_tip.stl" />
+                    </xacro:unless>
+                    <xacro:if value="${force_abs_paths}">
+                        <mesh filename="file://$(find robotiq_description)/meshes/collision/2f_85/left_finger_tip.stl" />
+                    </xacro:if>
                 </geometry>
                 <surface>
@@ -185,10 +266,20 @@
             <visual>
                 <geometry>
-                    <mesh filename="package://robotiq_description/meshes/visual/2f_85/right_finger_tip.dae" />
-                </geometry>
-            </visual>
-            <collision>
-                <geometry>
-                    <mesh filename="package://robotiq_description/meshes/collision/2f_85/right_finger_tip.stl" />
+                    <xacro:unless value="${force_abs_paths}">
+                        <mesh filename="package://robotiq_description/meshes/visual/2f_85/right_finger_tip.dae" />
+                    </xacro:unless>
+                    <xacro:if value="${force_abs_paths}">
+                        <mesh filename="file://$(find robotiq_description)/meshes/visual/2f_85/right_finger_tip.dae" />
+                    </xacro:if>
+                </geometry>
+            </visual>
+            <collision>
+                <geometry>
+                    <xacro:unless value="${force_abs_paths}">
+                        <mesh filename="package://robotiq_description/meshes/collision/2f_85/right_finger_tip.stl" />
+                    </xacro:unless>
+                    <xacro:if value="${force_abs_paths}">
+                        <mesh filename="file://$(find robotiq_description)/meshes/collision/2f_85/right_finger_tip.stl" />
+                    </xacro:if>
                 </geometry>
                 <surface>
